Commit message: Improve gameplay: stable robots, striker AI, and 5-goal match
- Load gazebo_ros_state plugin; fix controllers to use /gazebo/model_states
  and the SetEntityState service (ROS2 API)
- Rewrite robot_controller as a world-frame striker: get behind the ball and
  drive it toward the opponent goal, with per-robot randomized personality,
  situational pacing, slew-rate-smoothed velocity, opponent avoidance,
  stuck-escape, and a charge behavior to change the ball's direction
- Fix inverted goal assignment and guard against own-goals
- Stabilize robots: per-step planar_move, correct spawn height, lower COM,
  high roll/pitch inertia (un-tippable)
- Add first-to-5 match with in-Gazebo seven-segment scoreboard, game-over
  freeze, and reset of ball + both robots to kickoff after each goal

Co-Authored-By: Claude Opus 4.8 <noreply@anthropic.com>

File: src/humanoid_football/urdf/humanoid_robot.xacro (robot description, xacro)
@@ -37,9 +37,13 @@
       <origin xyz="0 0 0.05"/>
       <mass value="5.0"/>
-      <inertia
-        ixx="0.15"
+      <!-- Huge roll/pitch inertia (ixx, iyy) makes the body un-tippable:
+           planar_move sets velocity directly, so this does NOT affect driving,
+           but it makes contact impulses (robot-robot rams, ball hits) produce
+           negligible tilt before the plugin zeroes roll/pitch each step. -->
+      <inertia
+        ixx="100.0"
         ixy="0.0"
         ixz="0.0"
-        iyy="0.15"
+        iyy="100.0"
         iyz="0.0"
         izz="0.15"/>
@@ -62,12 +66,13 @@
     </collision>
     <inertial>
-      <mass value="1.0"/>
-      <inertia
-        ixx="0.01"
-        ixy="0"
-        ixz="0"
-        iyy="0.01"
-        iyz="0"
-        izz="0.01"/>
+      <!-- Light head keeps the center of mass low for stability -->
+      <mass value="0.4"/>
+      <inertia
+        ixx="0.004"
+        ixy="0"
+        ixz="0"
+        iyy="0.004"
+        iyz="0"
+        izz="0.004"/>
     </inertial>
   </link>
@@ -129,5 +134,5 @@
     </collision>
     <inertial>
-      <mass value="2.0"/>
+      <mass value="3.0"/>
       <inertia
         ixx="0.02"
@@ -194,5 +199,5 @@
     </collision>
     <inertial>
-      <mass value="2.0"/>
+      <mass value="3.0"/>
       <inertia
         ixx="0.02"
@@ -230,5 +235,8 @@
     <plugin name="${robot_name}_planar_move"
             filename="libgazebo_ros_planar_move.so">
-      <update_rate>50</update_rate>
+      <!-- Run every physics step (1 kHz). The plugin holds roll/pitch/z by
+           zeroing them each update; at a low rate the body drifts between
+           updates and topples, so this must match the physics rate. -->
+      <update_rate>1000</update_rate>
       <command_topic>cmd_vel</command_topic>
       <odometry_topic>odom</odometry_topic>
